Commit message: all working packages

File: betabot_description/urdf/betabot.urdf.xacro (robot description, xacro)
@@ -360,5 +360,5 @@
   <joint name="rplidar_joint" type="fixed">
     <axis xyz="0 1 0" />
-    <origin xyz="0 0 .109" rpy="0 0 0"/>
+    <origin xyz="0 0 .109" rpy="0 0 1.57"/>
     <parent link="base_link"/>
     <child link="rplidar_link"/>
